File: hardware/clinxer/potencia/FreeDS_potencia.kicad_pcb (KiCad board)
At the start: 2 copper layers, 61 x 93 mm, 16 parts, among them J1 Screw_Terminal_01x04, J2 Conn_01x04, Q3 BTA26-600BW, U1 MOC3041M, U5 Modulo de Control PWM de pote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

Commit message: Correcciones en arquitectura clinxer
Signed-off-by: Iván Sánchez Ortega <ivan@sanchezortega.es>
Parts:
- U5: value Modulo de Control PWM de potencia -> ~; footprint Module:YYAC-35 PWM TRIAC -> Module:YYAC-3S PWM TRIAC
- moved H1 1.11 mm to (171.4, 57.8)
Connections:
- Q3 pad 1: /Lin -> /A2_FUSE
- Q3 pad 2: /A2_FUSE -> /Lin
Routing:
- net /Lin: track 108.1 -> 118.1 mm
- net /A2_FUSE: track 31.7 -> 29.4 mm

Commit message: Corrección arq. clinxer: pines de optoacoplador
Signed-off-by: Iván Sánchez Ortega <ivan@sanchezortega.es>
Parts:
- moved TP1 11.0 mm to (142.2, 111.5)
- moved R2 4.20 mm to (142.2, 100.1)
Connections:
- R2 pad 1: /Lin -> /A2_FUSE
- R3 pad 1: /A2_FUSE -> /Lin
Routing:
- net /A2_FUSE: track 29.4 -> 49.3 mm
- net /Lin: track 118.1 -> 123.6 mm
- net /GND: track 50.5 -> 52.5 mm
- net /+5V: track 24.3 -> 22.3 mm
- net /N: track 76.5 -> 78.4 mm
- net Net-(Q3-G): track 105.7 -> 103.8 mm
- net /PWM: track 39.4 -> 40.2 mm, vias 1 -> 0
